Commit message: 

File: soccer_description/models/imu.xacro (robot description, xacro)
@@ -1,4 +1,4 @@
 <robot name="soccerbot" xmlns:xacro="http://www.ros.org/wiki/xacro">
-    <xacro:macro name="imu" params="origin">
+    <xacro:macro name="imu" params="origin imu_frame">
         <link name="imu_link" />
         <joint name="${origin}_imu" type="fixed">
@@ -16,5 +16,5 @@
                 <topic>__default_topic__</topic>
                 <plugin filename="libgazebo_ros_imu_sensor.so" name="imu_plugin">
-                    <topicName>imu</topicName>
+                    <topicName>imu_raw</topicName>
                     <bodyName>imu_link</bodyName>
                     <updateRateHZ>50.0</updateRateHZ>
@@ -22,5 +22,5 @@
                     <xyzOffset>0 0 0</xyzOffset>
                     <rpyOffset>0 0 0</rpyOffset>
-                    <frameName>imu_link</frameName>
+                    <frameName>${imu_frame}/imu_link</frameName>
                 </plugin>
                 <pose>0 0 0 0 0 0</pose>

File: soccer_description/models/robot.xacro (robot description, xacro)
@@ -34,5 +34,5 @@
         <leg name="right" origin="torso" direction="-1" />
         <head origin="torso" />
-        <imu origin="torso" />
+        <imu origin="torso" imu_frame="$(arg robot_name)" />
         <front_camera origin="head" />
         <gazebo>
